File: Dual-IO-Link-Master.sch (KiCad schematic (older format))
At the start: 56 parts, among them U20 MAX14819ATM+, U3 SI7421DN-T1-E3, U4 SI7421DN-T1-E3, U6 SI7421DN-T1-E3, U7 SI7421DN-T1-E3

Commit message: Imported and Started Footprint Associations
Parts:
- C42, C44, C51: footprint (none) -> CL10B105MO8NNWC:CL10B105MO8NNWC
- C43, C49: footprint (none) -> CL05A474KP5NNNC:CL05A474KP5NNNC
- C45, C46, C47, C48: footprint (none) -> CC0603JRNPO9BN271:CC0603JRNPO9BN271
- C50: footprint (none) -> CL10B104KB8NNNC:CL10B104KB8NNNC
- D27: footprint (none) -> LTSTC191KFKT:LTSTC191KFKT
- D28, D29: footprint (none) -> LTSTC191TBKT:LTSTC191TBKT
- D30, D31: footprint (none) -> LTSTC191KGKT:LTSTC191KGKT
- D32, D33: footprint (none) -> LTSTC191KRKT:LTSTC191KRKT
- U20: footprint 21-0144H_T4877-4_MXM -> MAX14819:MAX14819ATM&plus_
- U3, U4, U6, U7: footprint MOSFET_4DN-T1-E3_VIS -> SI7421DN-T1-E3:SI7421DN-T1-E3
Changed lines of the file:
@@
 F 0 "U20" H 5650 2500 60  0000 C CNN
 F 1 "MAX14819ATM+" H 5650 -100 60  0000 C CNN
-F 2 "21-0144H_T4877-4_MXM" H 5600 2640 60  0001 C CNN
+F 2 "MAX14819:MAX14819ATM&plus_" H 5600 2640 60  0001 C CNN
 F 3 "" H 4400 2400 60  0000 C CNN
 	1    4400 2400
@@
 F 0 "C51" H 7650 4350 50  0000 L CNN
 F 1 "1uF" H 7500 4150 50  0000 L CNN
-F 2 "" H 7688 4100 50  0001 C CNN
+F 2 "CL10B105MO8NNWC:CL10B105MO8NNWC" H 7688 4100 50  0001 C CNN
 F 3 "~" H 7650 4250 50  0001 C CNN
 	1    7650 4250
@@
 F 0 "C46" V 3500 3800 50  0000 L CNN
 F 1 "270pF" V 3600 4050 50  0000 L CNN
-F 2 "" H 3588 3850 50  0001 C CNN
+F 2 "CC0603JRNPO9BN271:CC0603JRNPO9BN271" H 3588 3850 50  0001 C CNN
 F 3 "~" H 3550 4000 50  0001 C CNN
 	1    3550 4000
@@
 F 0 "C44" V 3500 2700 50  0000 L CNN
 F 1 "1uF" V 3600 2950 50  0000 L CNN
-F 2 "" H 3588 2750 50  0001 C CNN
+F 2 "CL10B105MO8NNWC:CL10B105MO8NNWC" H 3588 2750 50  0001 C CNN
 F 3 "~" H 3550 2900 50  0001 C CNN
 	1    3550 2900
@@
 F 0 "C47" V 3500 4100 50  0000 L CNN
 F 1 "270pF" V 3600 4350 50  0000 L CNN
-F 2 "" H 3588 4150 50  0001 C CNN
+F 2 "CC0603JRNPO9BN271:CC0603JRNPO9BN271" H 3588 4150 50  0001 C CNN
 F 3 "~" H 3550 4300 50  0001 C CNN
 	1    3550 4300
@@
 F 0 "C45" V 3500 3550 50  0000 L CNN
 F 1 "270pF" V 3600 3750 50  0000 L CNN
-F 2 "" H 3588 3550 50  0001 C CNN
+F 2 "CC0603JRNPO9BN271:CC0603JRNPO9BN271" H 3588 3550 50  0001 C CNN
 F 3 "~" H 3550 3700 50  0001 C CNN
 	1    3550 3700
@@
 F 0 "C48" V 3500 4400 50  0000 L CNN
 F 1 "270pF" V 3600 4650 50  0000 L CNN
-F 2 "" H 3588 4450 50  0001 C CNN
+F 2 "CC0603JRNPO9BN271:CC0603JRNPO9BN271" H 3588 4450 50  0001 C CNN
 F 3 "~" H 3550 4600 50  0001 C CNN
 	1    3550 4600
@@
 F 0 "D28" H 1350 5700 50  0000 C CNN
 F 1 "BLUE" H 1350 5900 50  0000 C CNN
-F 2 "" H 1350 5800 50  0001 C CNN
+F 2 "LTSTC191TBKT:LTSTC191TBKT" H 1350 5800 50  0001 C CNN
 F 3 "~" H 1350 5800 50  0001 C CNN
 	1    1350 5800
@@
 F 0 "D29" H 1350 6000 50  0000 C CNN
 F 1 "BLUE" H 1350 6200 50  0000 C CNN
-F 2 "" H 1350 6100 50  0001 C CNN
+F 2 "LTSTC191TBKT:LTSTC191TBKT" H 1350 6100 50  0001 C CNN
 F 3 "~" H 1350 6100 50  0001 C CNN
 	1    1350 6100
@@
 F 0 "D30" H 1350 6300 50  0000 C CNN
 F 1 "GRN" H 1350 6500 50  0000 C CNN
-F 2 "" H 1350 6400 50  0001 C CNN
+F 2 "LTSTC191KGKT:LTSTC191KGKT" H 1350 6400 50  0001 C CNN
 F 3 "~" H 1350 6400 50  0001 C CNN
 	1    1350 6400
@@
 F 0 "D31" H 1350 6600 50  0000 C CNN
 F 1 "GRN" H 1350 6800 50  0000 C CNN
-F 2 "" H 1350 6700 50  0001 C CNN
+F 2 "LTSTC191KGKT:LTSTC191KGKT" H 1350 6700 50  0001 C CNN
 F 3 "~" H 1350 6700 50  0001 C CNN
 	1    1350 6700
@@
 F 0 "C49" V 3800 5050 50  0000 L CNN
 F 1 "0.47uF" V 3700 4700 50  0000 L CNN
-F 2 "" H 3788 4850 50  0001 C CNN
+F 2 "CL05A474KP5NNNC:CL05A474KP5NNNC" H 3788 4850 50  0001 C CNN
 F 3 "~" H 3750 5000 50  0001 C CNN
 	1    3750 5000
@@
 F 0 "C50" V 7700 3350 50  0000 L CNN
 F 1 "0.1uF" V 7600 3050 50  0000 L CNN
-F 2 "" H 7688 3150 50  0001 C CNN
+F 2 "CL10B104KB8NNNC:CL10B104KB8NNNC" H 7688 3150 50  0001 C CNN
 F 3 "~" H 7650 3300 50  0001 C CNN
 	1    7650 3300
@@
 F 0 "U21" V 8750 4100 60  0000 C CNN
 F 1 "SI7421DN-T1-E3" H 8800 3850 60  0000 C CNN
-F 2 "MOSFET_4DN-T1-E3_VIS" H 9150 4490 60  0001 C CNN
+F 2 "SI7421DN-T1-E3:SI7421DN-T1-E3" H 9150 4490 60  0001 C CNN
 F 3 "" H 8350 4250 60  0000 C CNN
 	1    8350 4250
@@
 F 0 "U22" V 8750 4600 60  0000 C CNN
 F 1 "SI7421DN-T1-E3" H 8800 4350 60  0000 C CNN
-F 2 "MOSFET_4DN-T1-E3_VIS" H 9150 4990 60  0001 C CNN
+F 2 "SI7421DN-T1-E3:SI7421DN-T1-E3" H 9150 4990 60  0001 C CNN
 F 3 "" H 8350 4750 60  0000 C CNN
 	1    8350 4750
@@
 F 0 "U19" V 3000 3600 60  0000 C CNN
 F 1 "SI7421DN-T1-E3" H 3050 3350 60  0000 C CNN
-F 2 "MOSFET_4DN-T1-E3_VIS" H 3400 3990 60  0001 C CNN
+F 2 "SI7421DN-T1-E3:SI7421DN-T1-E3" H 3400 3990 60  0001 C CNN
 F 3 "" H 2600 3750 60  0000 C CNN
 	1    2600 3750
@@
 F 0 "U18" V 3000 3100 60  0000 C CNN
 F 1 "SI7421DN-T1-E3" H 3050 2850 60  0000 C CNN
-F 2 "MOSFET_4DN-T1-E3_VIS" H 3400 3490 60  0001 C CNN
+F 2 "SI7421DN-T1-E3:SI7421DN-T1-E3" H 3400 3490 60  0001 C CNN
 F 3 "" H 2600 3250 60  0000 C CNN
 	1    2600 3250
@@
 F 0 "C43" V 3000 3650 50  0000 L CNN
 F 1 "0.47uF" V 2800 3400 50  0000 L CNN
-F 2 "" H 2988 3450 50  0001 C CNN
+F 2 "CL05A474KP5NNNC:CL05A474KP5NNNC" H 2988 3450 50  0001 C CNN
 F 3 "~" H 2950 3600 50  0001 C CNN
 	1    2950 3600
@@
 F 0 "C42" V 1550 2800 50  0000 L CNN
 F 1 "1uF" V 1550 2550 50  0000 L CNN
-F 2 "" H 1538 2600 50  0001 C CNN
+F 2 "CL10B105MO8NNWC:CL10B105MO8NNWC" H 1538 2600 50  0001 C CNN
 F 3 "~" H 1500 2750 50  0001 C CNN
 	1    1500 2750
@@
 F 0 "D32" H 1350 6900 50  0000 C CNN
 F 1 "RED" H 1350 7100 50  0000 C CNN
-F 2 "" H 1350 7000 50  0001 C CNN
+F 2 "LTSTC191KRKT:LTSTC191KRKT" H 1350 7000 50  0001 C CNN
 F 3 "~" H 1350 7000 50  0001 C CNN
 	1    1350 7000
@@
 F 0 "D33" H 1350 7200 50  0000 C CNN
 F 1 "RED" H 1350 7400 50  0000 C CNN
-F 2 "" H 1350 7300 50  0001 C CNN
+F 2 "LTSTC191KRKT:LTSTC191KRKT" H 1350 7300 50  0001 C CNN
 F 3 "~" H 1350 7300 50  0001 C CNN
 	1    1350 7300
@@
 F 0 "D27" H 1350 5400 50  0000 C CNN
 F 1 "ORNG" H 1350 5600 50  0000 C CNN
-F 2 "" H 1350 5500 50  0001 C CNN
+F 2 "LTSTC191KFKT:LTSTC191KFKT" H 1350 5500 50  0001 C CNN
 F 3 "~" H 1350 5500 50  0001 C CNN
 	1    1350 5500

Commit message: PCB/Footprint Work
Parts:
- removed TP37: L+A, symbol Connector:TestPoint
- removed TP38: L+B, symbol Connector:TestPoint
- removed TP39: DIA, symbol Connector:TestPoint
- removed TP42: DIB, symbol Connector:TestPoint
- removed TP44: LIA, symbol Connector:TestPoint
- removed TP45: LIB, symbol Connector:TestPoint
- removed TP46: CLKO, symbol Connector:TestPoint
- removed TP47: CLKI, symbol Connector:TestPoint
- removed TVS21, TVS22, TVS23, TVS24, TVS25, TVS26: SMCJ48A, SMCJSeries_LTF, symbol SMCJ48A:SMCJ48A
- added TVS21, TVS22, TVS23, TVS24, TVS25, TVS26: 48V, SMF48A:SMF48A, symbol Device:D_Zener
- D27: value ORNG -> IRQ
- D28: value BLUE -> LD1A
- D29: value BLUE -> LD2A
- D30: value GRN -> LD1B
- D31: value GRN -> LD2B
- D32: value RED -> L+A
- D33: value RED -> L+B
- R63, R64, R65, R66, R67: footprint (none) -> RC0603FR07820RL:RC0603FR07820RL
- R68, R69: footprint (none) -> RC0603FR076K8L:RC0603FR076K8L
- R70, R79: footprint (none) -> KRL1220E-M-R012-F-T5:KRL1220E-M-R012-F-T5
- R71, R72, R73, R74: footprint (none) -> RC0603JR07100RL:RC0603JR07100RL
- R75, R76, R77, R78: footprint (none) -> RC0603FR0710KL:RC0603FR0710KL
- TP40, TP41: footprint (none) -> RoboRIO-IO-Link-Master:TestPointFootprint
- TP43: value TP -> IRQ; footprint (none) -> RoboRIO-IO-Link-Master:TestPointFootprint
Connections:
- net CQA: now also TVS23.2 (A)
- net CQB: now also TVS26.2 (A)
- net DIA: now also TVS22.2 (A)
- net DIB: now also TVS25.2 (A)
- net GND: no longer U20.38 (A0), U20.39 (A1)
- net L+A: now also TVS21.2 (A)
- net L+B: now also TVS24.2 (A)
- net TVS_CLAMP: now also TVS21.1 (K), TVS22.1 (K), TVS23.1 (K), TVS24.1 (K), TVS25.1 (K), TVS26.1 (K)
- net *CS renamed MXP-CS
- net MISO renamed MXP-MISO
- net MOSI renamed MXP-MOSI
- net SCLK renamed MXP-SCLK
- new net A0: U20.38 (A0)
- new net A1: U20.39 (A1)
- no-connect marks 8 -> 10

Commit message: More PCB Layout
Parts:
- removed TP43: IRQ, RoboRIO-IO-Link-Master:TestPointFootprint, symbol Connector:TestPoint
