File: RoboRIO-IO-Link-Master.kicad_pcb (KiCad board)
At the start: 2 copper layers, 233 parts, among them J1 1885650000, J2 SFH11-PBPC-D17-ST-BK, J3 1885790000, J4 1885790000, M1 CSD18504Q5A, U1 SI4431BDY-T1-E3, U10 MAX14819ATM+, U11 SI7415DN-T1-E3, U12 SI7415DN-T1-E3, U13 SI7415DN-T1-E3, U14 SI7415DN-T1-E3, U15 MAX14819ATM+, U16 SI7415DN-T1-E3, U17 SI7415DN-T1-E3, U18 SI7415DN-T1-E3, U19 SI7415DN-T1-E3, U2 LM3488MMX_NOPB, U20 MAX14819ATM+, U21 SI7415DN-T1-E3, U22 SI7415DN-T1-E3, U3 SI7415DN-T1-E3, U4 SI7415DN-T1-E3, U5 MAX14819ATM+, U6 SI7415DN-T1-E3, U7 SI7415DN-T1-E3, U8 SI7415DN-T1-E3, U9 SI7415DN-T1-E3, Y1 ABM3B-14.7456MHZ-10-1-U-T

Commit message: More PCB Layout
Parts:
- removed TP10, TP21, TP32, TP43: IRQ, RoboRIO-IO-Link-Master:TestPointFootprint
- C10, C11, C13, C15, C17, C22, C23, C24, C25, C28, C29, C31, C4, R10, R11, R12, R13, R14, R15, R16, R17, R18, R19, R2, R28, R29, R3, R30, R31, R32, R33, R34, R35, R37, R38, R39, R40, R8, R9: moved to B.Cu
- U11, U12, U13, U14, U16, U17, U18, U19, U21, U22, U3, U4, U6, U7, U8, U9: value SI7415DN-T1-E3 -> SI7421DN-T1-E3
- moved R9 107.5 mm to (55.7, 140.1)
- moved D20 85.8 mm to (55.3, 83.4)
- moved D24 82.8 mm to (55.4, 88.6)
- moved D23 82.7 mm to (55.4, 86.0)
- moved D25 81.3 mm to (60.1, 83.3)
- moved TVS14 79.5 mm to (39.1, 109.1), turned to 180 degrees
- moved D22 78.6 mm to (55.4, 87.3)
- moved D21 78.6 mm to (55.4, 84.7)
- moved TVS11 77.2 mm to (44.9, 109.1), turned to 180 degrees
- moved D26 77.2 mm to (60.1, 84.6)
- moved TVS12 75.9 mm to (39.1, 111.9), turned to 180 degrees
- moved C27 74.1 mm to (46.0, 129.6), turned to 270 degrees
- moved R51 73.8 mm to (59.6, 87.7)
- moved R31 73.7 mm to (55.3, 126.1), turned to 180 degrees
- moved TVS16 72.0 mm to (56.0, 97.9)
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Connections:
- net MXP-DIO0 renamed Net-(J2-Pad11)
- C10 pad 1: /Dual IO-Link Master1/XO -> /Dual IO-Link Master4/XO
- C11 pad 2: /Dual IO-Link Master1/XI -> /Dual IO-Link Master4/XI
- C33 pad 2: /DL+6 -> /DL+0
- C35 pad 1: /DDI6 -> /DDI0
- C36 pad 1: /DCQ6 -> /DCQ0
- C37 pad 1: /DCQ7 -> /DCQ1
- C38 pad 1: /DDI7 -> /DDI1
- C39 pad 2: /DL+7 -> /DL+1
- C43 pad 2: /DL+0 -> /DL+6
- C45 pad 1: /DDI0 -> /DDI6
- C46 pad 1: /DCQ0 -> /DCQ6
- C47 pad 1: /DCQ1 -> /DCQ7
- C48 pad 1: /DDI1 -> /DDI7
- C49 pad 2: /DL+1 -> /DL+7
- D25 pad 2: /DL+6 -> /DL+0
- D26 pad 2: /DL+7 -> /DL+1
- D32 pad 2: /DL+0 -> /DL+6
- D33 pad 2: /DL+1 -> /DL+7
- R54 pad 2: /DL+6 -> /DL+0
- R55 pad 2: /DDI6 -> /DDI0
- R56 pad 2: /DDI7 -> /DDI1
- R57 pad 2: /DL+7 -> /DL+1
- R71 pad 2: /DL+0 -> /DL+6
- R72 pad 2: /DDI0 -> /DDI6
- R73 pad 2: /DDI1 -> /DDI7
- R74 pad 2: /DL+1 -> /DL+7
- R8 pad 2: /Dual IO-Link Master1/CLKI -> /Dual IO-Link Master4/CLKI
- TP29 pad 1: /DCQ6 -> /DCQ0
- TP30 pad 1: /DCQ7 -> /DCQ1
- TP40 pad 1: /DCQ0 -> /DCQ6
- TP41 pad 1: /DCQ1 -> /DCQ7
- TVS15 pad 2: /DL+6 -> /DL+0
- TVS16 pad 2: /DDI6 -> /DDI0
- TVS17 pad 2: /DCQ6 -> /DCQ0
- TVS18 pad 2: /DL+7 -> /DL+1
- TVS19 pad 2: /DDI7 -> /DDI1
- TVS20 pad 2: /DCQ7 -> /DCQ1
- TVS21 pad 2: /DL+0 -> /DL+6
- TVS22 pad 2: /DDI0 -> /DDI6
- TVS23 pad 2: /DCQ0 -> /DCQ6
- TVS24 pad 2: /DL+1 -> /DL+7
- TVS25 pad 2: /DDI1 -> /DDI7
- TVS26 pad 2: /DCQ1 -> /DCQ7
- U10 pad 44: /Dual IO-Link Master4/CLKI -> /Dual IO-Link Master1/CLKI
- U14 pad 5: /DL+6 -> /DL+0
- U14 pad 6: /DL+6 -> /DL+0
- U14 pad 7: /DL+6 -> /DL+0
- U14 pad 8: /DL+6 -> /DL+0
- U15 pad 17: /DCQ6 -> /DCQ0
- U15 pad 20: /DCQ7 -> /DCQ1
- U15 pad 38: +3V3 -> GND
- U15 pad 39: +3V3 -> GND
- U15 pad 44: /Dual IO-Link Master4/CLKO -> /Dual IO-Link Master2/CLKI
- U17 pad 5: /DL+7 -> /DL+1
- U17 pad 6: /DL+7 -> /DL+1
- U17 pad 7: /DL+7 -> /DL+1
- U17 pad 8: /DL+7 -> /DL+1
- U19 pad 5: /DL+0 -> /DL+6
- U19 pad 6: /DL+0 -> /DL+6
- U19 pad 7: /DL+0 -> /DL+6
- U19 pad 8: /DL+0 -> /DL+6
- U20 pad 17: /DCQ0 -> /DCQ6
- U20 pad 20: /DCQ1 -> /DCQ7
- U20 pad 38: GND -> +3V3
- U20 pad 39: GND -> +3V3
- U20 pad 44: /Dual IO-Link Master2/CLKI -> /Dual IO-Link Master1/CLKO
- U22 pad 5: /DL+1 -> /DL+7
- U22 pad 6: /DL+1 -> /DL+7
- U22 pad 7: /DL+1 -> /DL+7
- U22 pad 8: /DL+1 -> /DL+7
- Y1 pad 1: /Dual IO-Link Master1/XO -> /Dual IO-Link Master4/XO
- Y1 pad 3: /Dual IO-Link Master1/XI -> /Dual IO-Link Master4/XI
Routing:
- net TVS_CLAMP: track 7.05 -> 119.2 mm, vias 0 -> 3
- net MXP-MOSI: track 0.00 -> 95.5 mm, vias 0 -> 6
- net MXP-MISO: track 0.00 -> 93.3 mm, vias 0 -> 6
- net MXP-SCLK: track 0.00 -> 89.2 mm, vias 0 -> 6
- net MXP-CS: track 0.00 -> 85.9 mm, vias 0 -> 4
- net /DL+3: track 12.7 -> 74.4 mm, vias 0 -> 3
- net /DL+4: track 5.00 -> 65.0 mm, vias 0 -> 2
- net /DDI4: track 5.00 -> 64.7 mm, vias 0 -> 1
- net /DL+0: track 5.00 -> 59.7 mm, vias 0 -> 1
- net /DCQ4: track 5.00 -> 59.5 mm, vias 0 -> 2
- net /DL+2: track 5.00 -> 58.4 mm, vias 0 -> 2
- net /DCQ0: track 5.00 -> 57.3 mm, vias 0 -> 1
- net /DDI0: track 5.00 -> 55.6 mm, vias 0 -> 1
- net /DDI5: track 5.00 -> 51.0 mm, vias 0 -> 2
- net /DCQ7: track 5.00 -> 49.5 mm, vias 0 -> 1
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Other:
- net class Default: clearance 0.2 -> 0.1524; trace_width 0.25 -> 0.254; via_dia 0.8 -> 0.635; via_drill 0.4 -> 0.3048
- rule trace_clearance: 0.2 -> 0.1524

Commit message: Wrapping up first prototype
Parts:
- added G***: LOGO, RoboRIO-IO-Link-Master:34e, F.Cu at (45.5, 112.2)
- added G***: LOGO, RoboRIO-IO-Link-Master:rr, F.Cu at (45.5, 100.0)
- added G***: LOGO, RoboRIO-IO-Link-Master:io-link, F.Cu at (45.5, 106.2)
- added R80: 1k, RC0603FR071KL:RC0603FR071KL, F.Cu at (66.4, 118.0)
- added R81: 1k, RC0603FR071KL:RC0603FR071KL, B.Cu at (51.9, 112.9)
- added R82: 1k, RC0603FR071KL:RC0603FR071KL, F.Cu at (45.9, 96.2)
- C31: moved to F.Cu
- C32, C33, C34, C35, C36, C37, C38, C39, C43, C44, C45, C46, C48, C49, R36, R46, R47, R48, R49, R50, R51, R52, R53, R63, R64, R65, R66, R67, R68, R69, R70, R73, R74, R75, R76, R77, R78, R79: moved to B.Cu
- moved R50 46.9 mm to (55.3, 88.4), turned to 180 degrees
- moved R46 46.8 mm to (55.3, 82.5), turned to 180 degrees
- moved TP40 46.6 mm to (41.8, 84.4)
- moved TP41 45.6 mm to (40.7, 82.8)
- moved R49 43.8 mm to (55.3, 85.4), turned to 180 degrees
- moved R47 43.7 mm to (55.3, 83.9), turned to 180 degrees
- moved R48 43.7 mm to (55.3, 86.9), turned to 180 degrees
- moved R67 43.6 mm to (55.3, 95.7), turned to 180 degrees
- moved R65 42.8 mm to (55.3, 94.3), turned to 180 degrees
- moved R63 42.6 mm to (55.3, 89.8), turned to 180 degrees
- moved R66 42.3 mm to (55.3, 92.8), turned to 180 degrees
- moved R64 42.0 mm to (55.3, 91.3), turned to 180 degrees
- moved TP29 37.3 mm to (60.4, 81.5)
- moved R45 35.5 mm to (50.7, 128.5), turned to 180 degrees
- moved C40 35.5 mm to (62.8, 95.4), turned to 180 degrees
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Connections:
- U10 pad 44: /Dual IO-Link Master1/CLKI -> /Dual IO-Link Master3/CLKO
- U15 pad 44: /Dual IO-Link Master2/CLKI -> /Dual IO-Link Master4/CLKO
- U5 pad 44: /Dual IO-Link Master3/CLKI -> /Dual IO-Link Master2/CLKO
Routing:
- net +24V: track 65.8 -> 456.3 mm, vias 9 -> 22
- net +3V3: track 3.15 -> 178.0 mm, vias 0 -> 16
- net GND: track 4.85 -> 168.9 mm, vias 0 -> 688
- net +5V: track 6.64 -> 144.3 mm, vias 1 -> 8
- net /DL+7: track 44.8 -> 83.9 mm, vias 0 -> 1
- net /DCQ1: track 9.31 -> 48.4 mm, vias 0 -> 2
- net /DDI1: track 8.64 -> 46.9 mm, vias 0 -> 2
- net /DL+1: track 10.0 -> 46.7 mm, vias 0 -> 2
- net /DDI7: track 11.4 -> 46.7 mm, vias 0 -> 2
- net Net-(C6-Pad1): track 5.38 -> 40.3 mm, vias 0 -> 3
- net /DL+6: track 19.1 -> 53.3 mm, vias 1 -> 3
- net /Dual IO-Link Master4/#RDYB-LD1B: track 0.00 -> 32.6 mm, vias 0 -> 1
- net /Dual IO-Link Master4/#ERRB-LD2B: track 0.00 -> 32.1 mm, vias 0 -> 1
- net /Dual IO-Link Master3/CLKO: track 0.00 -> 30.5 mm
- net /Dual IO-Link Master4/#RDYA-LD1A: track 0.00 -> 30.3 mm, vias 0 -> 1
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- added copper zone on B.Cu, net GND
- added copper zone on F.Cu, net GND
Other:
- board outline added: 56.6 x 77.5 mm
- board text added: "Liam Snow"
- board text added: "RoboRIO IO-Link Board"

Commit message: tweaking
Parts:
- U11, U12, U13, U14, U16, U17, U18, U19, U21, U22, U3, U4, U6, U7, U8, U9: value SI7421DN-T1-E3 -> SI7415DN-T1-E3
Routing:
- net /DL+7: track 83.9 -> 84.6 mm
- net +24V: track 456.3 -> 456.9 mm
- net GND: vias 688 -> 662
